File: ADS1X15/ADS1X15.kicad_pcb (KiCad board)
At the start: 2 copper layers, 17.5 x 22.6 mm, 20 parts, among them J1 Conn_01x05, J2 Conn_01x05

Commit message: ADS1X15 Added in place of ADS1015 and ADS1115
Parts:
- removed ADS1015: ADS1015IDGS, Package_SO:TSSOP-10_3x3mm_P0.5mm
- added ADS1X15: ADS1115IDGS, Package_SO:TSSOP-10_3x3mm_P0.5mm, F.Cu at (65.5, 38.5)
- G***: footprint logo:SirBoard71X22 -> logo:SirBoard79x25
- moved G*** 0.25 mm to (65.5, 29.3)
Other:
- board text added: "12 Bit 16 Bit"
- board text added: "ADS1X15"
- board text added: "www.SirBoard.com"
- board text removed: "ADS1015 4 Channel 12 Bit ADC"
