File: ADXL32X/ADXL32X.sch (KiCad schematic (older format))
At the start: 13 parts, among them J1 Conn_01x04, J2 Conn_01x04, U1 AP2127K-3.3, U2 ADXL32X

Commit message: Schematic PDF and 3D Renders added
Parts:
- U2: symbol ADXL32X:ADXL327 -> ADXL32X-rescue:ADXL327-ADXL32X
Changed lines of the file:
@@
 EESchema Schematic File Version 4
-LIBS:ADXL327-cache
+LIBS:ADXL32X-cache
 EELAYER 29 0
 EELAYER END
@@
 $EndComp
 $Comp
-L ADXL32X:ADXL327 U2
+L ADXL32X-rescue:ADXL327-ADXL32X U2
 U 1 1 5DF1EFC3
 P 1400 1150

Commit message: Part numbers added for all variants
Parts:
- U2: Part (none) -> C208133; C207396; 759-1998; 709-0136; 709-0145
Changed lines of the file:
@@
 F 2 "Package_DFN_QFN:QFN-16-1EP_4x4mm_P0.65mm_EP2.1x2.1mm" H 1400 1725 50  0001 C CNN
 F 3 "" H 1400 1725 50  0001 C CNN
+F 4 "C208133; C207396; 759-1998; 709-0136; 709-0145" H 1400 1150 50  0001 C CNN "Part"
 	1    1400 1150
 	1    0    0    -1
